Commit message: Clean up kinova urdf - comment out unneeded links

File: assets/kortex_description/robots/gen3_robotiq_2f_85.urdf (robot description, URDF)
Before this commit: robot gen3_robotiq_2f_85, 28 links, 27 joints
Links:
- removed link realsense_camera
- removed link realsense_camera_mount
- link base_link: geometry collision mesh filename=package://kortex_description/arms/gen3/7dof/meshes/base_lin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; visual mesh filename=package://kortex_description/arms/gen3/7dof/meshes/base_lin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
- link bracelet_link: geometry collision mesh filename=package://kortex_description/arms/gen3/7dof/meshes/bracelet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; visual mesh filename=package://kortex_description/arms/gen3/7dof/meshes/bracelet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
- link camera_depth_frame: geometry visual box size=0.005 0.005 0.005
- link forearm_link: geometry collision mesh filename=package://kortex_description/arms/gen3/7dof/meshes/forearm_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; visual mesh filename=package://kortex_description/arms/gen3/7dof/meshes/forearm_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
- link half_arm_1_link: geometry collision mesh filename=package://kortex_description/arms/gen3/7dof/meshes/half_arm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; visual mesh filename=package://kortex_description/arms/gen3/7dof/meshes/half_arm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
- link half_arm_2_link: geometry collision mesh filename=package://kortex_description/arms/gen3/7dof/meshes/half_arm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; visual mesh filename=package://kortex_description/arms/gen3/7dof/meshes/half_arm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
- link left_inner_finger: geometry collision mesh filename=package://kortex_description/grippers/robotiq_2f_85/meshes/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 scale=0.001 0.001 0.001; visual mesh filename=package://kortex_description/grippers/robotiq_2f_85/meshes/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 scale=0.001 0.001 0.001
- link left_inner_knuckle: geometry collision mesh filename=package://kortex_description/grippers/robotiq_2f_85/meshes/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 scale=0.001 0.001 0.001; visual mesh filename=package://kortex_description/grippers/robotiq_2f_85/meshes/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 scale=0.001 0.001 0.001
- link left_outer_finger: geometry collision mesh filename=package://kortex_description/grippers/robotiq_2f_85/meshes/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 scale=0.001 0.001 0.001; visual mesh filename=package://kortex_description/grippers/robotiq_2f_85/meshes/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 scale=0.001 0.001 0.001
- link left_outer_knuckle: geometry collision mesh filename=package://kortex_description/grippers/robotiq_2f_85/meshes/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 scale=0.001 0.001 0.001; visual mesh filename=package://kortex_description/grippers/robotiq_2f_85/meshes/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 scale=0.001 0.001 0.001
- link right_inner_finger: geometry collision mesh filename=package://kortex_description/grippers/robotiq_2f_85/meshes/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 scale=0.001 0.001 0.001; visual mesh filename=package://kortex_description/grippers/robotiq_2f_85/meshes/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 scale=0.001 0.001 0.001
- link right_inner_knuckle: geometry collision mesh filename=package://kortex_description/grippers/robotiq_2f_85/meshes/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 scale=0.001 0.001 0.001; visual mesh filename=package://kortex_description/grippers/robotiq_2f_85/meshes/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 scale=0.001 0.001 0.001
- link right_outer_finger: geometry collision mesh filename=package://kortex_description/grippers/robotiq_2f_85/meshes/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 scale=0.001 0.001 0.001; visual mesh filename=package://kortex_description/grippers/robotiq_2f_85/meshes/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 scale=0.001 0.001 0.001
- link right_outer_knuckle: geometry collision mesh filename=package://kortex_description/grippers/robotiq_2f_85/meshes/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 scale=0.001 0.001 0.001; visual mesh filename=package://kortex_description/grippers/robotiq_2f_85/meshes/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 scale=0.001 0.001 0.001
- link robotiq_arg2f_base_link: geometry collision mesh filename=package://kortex_description/grippers/robotiq_2f_85/meshes/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; visual mesh filename=package://kortex_description/grippers/robotiq_2f_85/meshes/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 scale=0.001 0.001 0.001
- link shoulder_link: geometry collision mesh filename=package://kortex_description/arms/gen3/7dof/meshes/shoulder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; visual mesh filename=package://kortex_description/arms/gen3/7dof/meshes/shoulder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
- link spherical_wrist_1_link: geometry collision mesh filename=package://kortex_description/arms/gen3/7dof/meshes/spherica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; visual mesh filename=package://kortex_description/arms/gen3/7dof/meshes/spherica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
- link spherical_wrist_2_link: geometry collision mesh filename=package://kortex_description/arms/gen3/7dof/meshes/spherica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; visual mesh filename=package://kortex_description/arms/gen3/7dof/meshes/spherica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
Joints:
- removed joint joint_realsense_camera
- removed joint joint_realsense_camera_mount
- joint depth_module: origin xyz=0.0275 0.066 -0.00305 rpy=3.14159265358979 3.14159265358979 0 -> xyz=0.0175 0.061 0.03 rpy=0 -1.57 0
